File: Beating Heart.brd (EAGLE design)
At the start: 49.6 x 46.4 mm, 26 parts, among them U2 ATTINY85

Commit message: adds updates to board and schematic
Parts:
- moved S3 4.02 mm to (39.4, 39.4)
Connections:
- new net VBAT: S3.1, U$1.+$1
- net VCC: no longer S3.1, U$1.+$1
Routing:
- net VCC: track 207.0 -> 180.6 mm
- net VBAT: track 0.00 -> 14.7 mm
